File: kc1fsz-rx7.kicad_sch (KiCad schematic)
At the start: 18 parts, among them J1 IQ, J2 Power, J3 Config, J4 Conn_01x06, U1 PCM1804DBR

Commit message: Added docs
Other:
- company: (none) -> Bruce MacKinnon KC1FSZ
- title: (none) -> PCM1804 Breakout Board
Changed lines of the file:
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@@
 	(generator_version "8.0")
 	(paper "A4")
+	(title_block
+		(title "PCM1804 Breakout Board")
+		(date "2024-12-03")
+		(rev "1")
+		(company "Bruce MacKinnon KC1FSZ")
+	)
 	(junction
 		(at 93.98 118.11)
